File: ComAir-eval.kicad_sch (KiCad schematic)
At the start: 38 parts, among them J1 Conn_01x05, J101 Conn_01x02, J102 Conn_01x02, J103 Conn_01x01, J104 Conn_01x01, J105 Conn_01x07, J106 Conn_01x06, J107 Conn_01x06, SW101 SW_Push, SW102 SW_Push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

Commit message: Set release number to 1.1
Signed-off-by: Alexis Jeandet <alexis.jeandet@member.fsf.org>
Other:
- company: (none) -> LPP/CNRS
- title: (none) -> ComAir-Eval
