File: Power.kicad_sch (KiCad schematic)
At the start: 19 parts, among them U201 SPV1050TTR

Commit message: Set release number to 1.1
Signed-off-by: Alexis Jeandet <alexis.jeandet@member.fsf.org>
Parts:
- R201: value R -> 10M
- R202: value R -> 3M
- R203: value R -> 680k
- R204: value R -> 2.7M
- R205: value R -> 6.2M
- R208: value R -> 500k
Other:
- company: (none) -> LPP/CNRS
- title: (none) -> ComAir-Eval
