File: Sensor.kicad_sch (KiCad schematic)
At the start: 9 parts, among them U1 TS3A24159DGSR, U2 SCD41

Commit message: Set release number to 1.1
Signed-off-by: Alexis Jeandet <alexis.jeandet@member.fsf.org>
Connections:
- net 3.3V: now also U1.1 (VCC), U1.10; no longer U1.2
- net 3V3_SCD: now also U1.9; no longer U1.3
- net GND: now also U1.6 (GND), U1.7; no longer U1.5
- net POWER_EN: now also U1.8; no longer U1.4
Other:
- company: (none) -> LPP/CNRS
- title: (none) -> ComAir-Eval
