File: USB.kicad_sch (KiCad schematic)
At the start: 17 parts, among them J401 DX07S016JA1R1500, U301 MCP73831-2-OT, U401 NCP718xSN330, U402 TPD2E2U06

Commit message: Set release number to 1.1
Signed-off-by: Alexis Jeandet <alexis.jeandet@member.fsf.org>
Other:
- company: (none) -> LPP/CNRS
- title: (none) -> ComAir-Eval
